File: sch/main/main.kicad_sch (KiCad schematic)
At the start: 7 parts, among them J1 Micro_SD_Card, U1 CH340E, U2 240X240_IPS, U3 PSRAM64H, U4 STC15W104

Commit message: Add sd test.
Connections:
- net MISO: now also U4.8 (P3.3); no longer U4.16 (P3.3)
- net MOSI: now also U4.7 (P3.2); no longer U4.15 (P3.2)
- net RXD: now also U4.5 (P3.0); no longer U4.13 (P3.0)
- net TXD: now also U4.6 (P3.1); no longer U4.14 (P3.1)
Changed lines of the file:
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@@
     )
     (pin "1")
-    (pin "13")
-    (pin "14")
-    (pin "15")
-    (pin "16")
     (pin "2")
     (pin "3")
     (pin "4")
+    (pin "5")
+    (pin "6")
+    (pin "7")
+    (pin "8")
   )
   (symbol (lib_id "power:GND") (at 118.11 83.82 0) (unit 1)

Commit message: Add mini-rv32ima
Parts:
- added D2: LED, symbol Device:LED
- added R2: 1K, symbol Device:R
Connections:
- net GND: now also D2.1 (K)
- net TXD: now also R2.2
- new net: D2.2 (A), R2.1
Changed lines of the file:
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@@
+    )
+  )
+  (global_label "TXD" (shape input) (at 215.9 106.68 90) (fields_autoplaced)
+    (effects (font (size 1.27 1.27)) (justify left))
+    (property "Intersheet References" "${INTERSHEET_REFS}" (id 0) (at 215.8206 100.8198 90)
+      (effects (font (size 1.27 1.27)) (justify left) hide)
     )
   )
@@
     (pin "1")
   )
+  (symbol (lib_id "power:GND") (at 215.9 121.92 0) (unit 1)
+    (in_bom yes) (on_board yes) (fields_autoplaced)
+    (property "Reference" "#PWR08" (id 0) (at 215.9 128.27 0)
+      (effects (font (size 1.27 1.27)) hide)
+    )
+    (property "Value" "GND" (id 1) (at 215.9 127 0))
+    (property "Footprint" "" (id 2) (at 215.9 121.92 0)
+      (effects (font (size 1.27 1.27)) hide)
+    )
+    (property "Datasheet" "" (id 3) (at 215.9 121.92 0)
+      (effects (font (size 1.27 1.27)) hide)
+    )
+    (pin "1")
+  )
   (symbol (lib_id "power:GND") (at 196.85 107.95 0) (unit 1)
     (in_bom yes) (on_board yes) (fields_autoplaced)
@@
     (pin "8")
   )
+  (symbol (lib_id "Device:LED") (at 215.9 118.11 90) (unit 1)
+    (in_bom yes) (on_board yes) (fields_autoplaced)
+    (property "Reference" "D2" (id 0) (at 219.71 118.4274 90)
+      (effects (font (size 1.27 1.27)) (justify right))
+    )
+    (property "Value" "LED" (id 1) (at 219.71 120.9674 90)
+      (effects (font (size 1.27 1.27)) (justify right))
+    )
+    (property "Footprint" "" (id 2) (at 215.9 118.11 0)
+      (effects (font (size 1.27 1.27)) hide)
+    )
+    (property "Datasheet" "~" (id 3) (at 215.9 118.11 0)
+      (effects (font (size 1.27 1.27)) hide)
+    )
+    (pin "1")
+    (pin "2")
+  )
   (symbol (lib_id "power:GND") (at 128.27 121.92 0) (unit 1)
     (in_bom yes) (on_board yes) (fields_autoplaced)
-    (property "Reference" "#PWR?" (id 0) (at 128.27 128.27 0)
+    (property "Reference" "#PWR09" (id 0) (at 128.27 128.27 0)
       (effects (font (size 1.27 1.27)) hide)
     )
@@
     (pin "8")
     (pin "9")
+  )
+  (symbol (lib_id "Device:R") (at 215.9 110.49 180) (unit 1)
+    (in_bom yes) (on_board yes) (fields_autoplaced)
+    (property "Reference" "R2" (id 0) (at 218.44 109.2199 0)
+      (effects (font (size 1.27 1.27)) (justify right))
+    )
+    (property "Value" "1K" (id 1) (at 218.44 111.7599 0)
+      (effects (font (size 1.27 1.27)) (justify right))
+    )
+    (property "Footprint" "" (id 2) (at 217.678 110.49 90)
+      (effects (font (size 1.27 1.27)) hide)
+    )
+    (property "Datasheet" "~" (id 3) (at 215.9 110.49 0)
+      (effects (font (size 1.27 1.27)) hide)
+    )
+    (pin "1")
+    (pin "2")
   )
   (symbol (lib_id "Device:R") (at 101.6 82.55 180) (unit 1)
@@
       (reference "#PWR07") (unit 1) (value "GND") (footprint "")
     )
+    (path "/8710fbe1-4bc6-40b8-9ae5-fd396f460a5b"
+      (reference "#PWR08") (unit 1) (value "GND") (footprint "")
+    )
     (path "/cb7fc3dd-c3e8-474b-a78e-76fe86c074fc"
-      (reference "#PWR?") (unit 1) (value "GND") (footprint "")
+      (reference "#PWR09") (unit 1) (value "GND") (footprint "")
     )
     (path "/4da8687a-b41a-4997-a7c7-072e3068aef7"
       (reference "D1") (unit 1) (value "LED") (footprint "")
     )
+    (path "/c220786d-2db5-4b8f-8e46-970446d95add"
+      (reference "D2") (unit 1) (value "LED") (footprint "")
+    )
     (path "/d5d9204f-9197-4e2c-9321-344189dcf077"
       (reference "J1") (unit 1) (value "Micro_SD_Card") (footprint "")
@@
       (reference "R1") (unit 1) (value "1K") (footprint "")
     )
+    (path "/d7305eec-79b8-4ec6-84c1-11c7db800378"
+      (reference "R2") (unit 1) (value "1K") (footprint "")
+    )
     (path "/4b7d5d94-5daa-49c5-89d9-7d989a6027e2"
